File: hardware/neopico-hd/neopico-hd.kicad_sch (KiCad schematic)
At the start: 9 parts, among them U1 SN74LVC2G14DBV, U2 SN74LVC2G14DBV, U3 SN74LVC245APW, U4 SN74LVC245APW

Commit message: ?
Parts:
- added C5: 0.1u, custom_components:SM0603_Capa_libcms, symbol Device:C
- added J1: HDMI_A, symbol Connector:HDMI_A
- added U5: SN74LVC245APW, Package_SO:TSSOP-20_4.4x6.5mm_P0.65mm, symbol Logic_LevelTranslator:SN74LVC245APW
Connections:
- net GND: now also U3.1 (DIR), U4.1 (DIR), C5.2, J1.17 (GND), U5.1 (DIR), U5.10 (GND)
- net VCC: now also C5.1, U5.20 (VCC)
- net +3V3: now reaches U4.19 (~{OE})
- net +3V3: now also U3.19 (~{OE}), U5.19 (~{OE})
- net +5V: now reaches A1.1 (VBUS)
- net +5V: now also J1.18 (+5V)
- net HDMI_CLK_N: now reaches A1.18 (GPIO12)
- net HDMI_CLK_N: now also J1.12 (CK-)
- net HDMI_CLK_P: now reaches A1.19 (GPIO13)
- net HDMI_CLK_P: now also J1.10 (CK+)
- net HTMI_D0_N: now reaches A1.20 (GPIO14)
- net HTMI_D0_N: now also J1.9 (D0-)
- net HTMI_D0_P: now reaches A1.21 (GPIO15)
- net HTMI_D0_P: now also J1.7 (D0+)
- net HTMI_D1_N: now reaches A1.22 (GPIO16)
- net HTMI_D1_N: now also J1.6 (D1-)
- net HTMI_D1_P: now reaches A1.23 (GPIO17)
- net HTMI_D1_P: now also J1.4 (D1+)
- net HTMI_D2_N: now reaches A1.24 (GPIO18)
- net HTMI_D2_N: now also J1.3 (D2-)
- net HTMI_D2_P: now reaches A1.25 (GPIO19)
- net HTMI_D2_P: now also J1.1 (D2+)
- new net DAT: U5.18 (B1)
- new net MVS_DAT: U5.2 (A1)
- new net MVS_WS: U5.3 (A2)
- new net WS: U5.17 (B2)
- no-connect marks 0 -> 24
Other:
- moved on the sheet: A1, C2, U1
