File: hardware/neopico-hd/neopico-hd.kicad_sch (KiCad schematic)
At the start: 19 parts, among them J1 HDMI_A, U1 SN74LVC2G14DBV, U2 SN74LVC2G14DBV, U3 SN74LVC245APW, U4 SN74LVC245APW, U5 SN74LVC245APW, U6 ESD224DQA, U7 ESD224DQA

Commit message: Update hardware project
Parts:
- A1: footprint (none) -> Module:WeAct_RP2350B
- renumbered C4 to C3, C3 to C4
Connections:
- net GND: now also U6.3 (VSS), U6.8 (VSS), U7.3 (VSS), U7.8 (VSS)
Other:
- note added: "Power Input"
- note removed: "Power"
- moved on the sheet: C2, C6, C7, D1, F1, FB1, J1, U1, U6, U7
