File: hardware/neopico-hd/neopico-hd.kicad_sch (KiCad schematic)
At the start: 25 parts, among them J1 HDMI_A, J2 Conn_02x05_Top_Bottom, J3 Conn_02x05_Top_Bottom, J4 Audio, U1 A_BUFF, U11 74LVC2G17, U2 V_BUFF, U3 RG_LVS, U4 GB_LVS, U5 AV_LVS, U6 V_BUFF, U7 74LVC2G17, U9 SN74LVC2G14DBV

Commit message: Update PCB
Parts:
- removed C8: 0.1u, Capacitor_SMD:C_0805_2012Metric_Pad1.18x1.45mm_HandSolder, symbol Device:C
- removed J3: Conn_02x05_Top_Bottom, Connector_IDC:IDC-Header_2x05_P2.54mm_Vertical, symbol Connector_Generic:Conn_02x05_Top_Bottom
- removed U11: 74LVC2G17, Package_TO_SOT_SMD:TSOT-23-6_HandSoldering, symbol neopico-hd:74LVC2G17
- removed U6: V_BUFF, Package_TO_SOT_SMD:SOT-23-6, symbol 74xGxx:SN74LVC2G14DBV
- removed U7: 74LVC2G17, symbol 74xGxx:74LVC2G17
- removed U9: SN74LVC2G14DBV, Package_TO_SOT_SMD:SOT-23-6, symbol 74xGxx:SN74LVC2G14DBV
- added J3: Audio, Connector_JST:JST_XA_B03B-XASK-1_1x03_P2.50mm_Vertical, symbol Connector_Generic:Conn_01x03
- added J5: AUX, Connector_JST:JST_XA_B08B-XASK-1_1x08_P2.50mm_Vertical, symbol Connector:Conn_01x08_Socket
- added J6: Conn_01x02_Pin, Connector_PinHeader_2.54mm:PinHeader_1x02_P2.54mm_Vertical, symbol Connector:Conn_01x02_Pin
- J2: footprint Connector_IDC:IDC-Header_2x05_P2.54mm_Vertical -> Connector_IDC:IDC-Header_2x10_P2.54mm_Vertical; symbol Connector_Generic:Conn_02x05_Top_Bottom -> Connector_Generic:Conn_02x10_Odd_Even
Connections:
- net +3V3: now also A1.56 (3V3)
- net B0: now also A1.39 (GPIO33); no longer A1.43 (GPIO37)
- net B1: now also A1.38 (GPIO32); no longer A1.42 (GPIO36)
- net B2: now also A1.37 (GPIO31); no longer A1.41 (GPIO35)
- net B3: now also A1.36 (GPIO30); no longer A1.40 (GPIO34)
- net B4: now also A1.35 (GPIO29); no longer A1.39 (GPIO33)
- net CSYNC: now also A1.33 (GPIO27), U2.6 (1Y); no longer A1.36 (GPIO30), U2.4 (2Y)
- net DARK: now also A1.51 (GPIO45), U5.11 (B8); no longer A1.38 (GPIO32)
- net G0: now also A1.44 (GPIO38); no longer A1.48 (GPIO42)
- net G1: now also A1.43 (GPIO37); no longer A1.47 (GPIO41)
- net G2: now also A1.42 (GPIO36); no longer A1.46 (GPIO40)
- net G3: now also A1.41 (GPIO35); no longer A1.45 (GPIO39)
- net G4: now also A1.40 (GPIO34); no longer A1.44 (GPIO38)
- net GND: now also A1.3 (AGND), A1.4 (AGND), A1.57 (AGND), A1.59 (AGND), A1.60 (AGND), J6.1 (Pin_1); no longer A1.61 (AGND)
- net MVS_B0: now also J2.11 (Pin_11)
- net MVS_B1: now also J2.12 (Pin_12)
- net MVS_B2: now also J2.13 (Pin_13)
- net MVS_B3: now also J2.14 (Pin_14)
- net MVS_B4: now also J2.15 (Pin_15)
- net MVS_CSYNC: now also J2.18 (Pin_18), U2.1 (1A); no longer U2.3 (2A)
- net MVS_DARK: now also J2.17 (Pin_17), U5.9 (A8)
- net MVS_PCKL: now also J2.19 (Pin_19), U2.3 (2A); no longer U2.1 (1A)
- net MVS_SHD: now also J2.16 (Pin_16), U5.8 (A7)
- net PCKL: now also A1.34 (GPIO28), U2.4 (2Y); no longer A1.35 (GPIO29), U2.6 (1Y)
- net R0: now also A1.49 (GPIO43); no longer A1.54 (GPIO47)
- net R1: now also A1.48 (GPIO42); no longer A1.53 (GPIO46)
- net R2: now also A1.47 (GPIO41); no longer A1.52 (GPIO45)
- net R3: now also A1.46 (GPIO40); no longer A1.51 (GPIO44)
- net R4: now also A1.45 (GPIO39); no longer A1.50 (GPIO43)
- net SHD: now also A1.50 (GPIO44), U5.12 (B7); no longer A1.37 (GPIO31)
- net at A1.10 (GPIO4): now also J5.2 (Pin_2)
- net at A1.11 (GPIO5): now also J5.3 (Pin_3)
- net at A1.12 (GPIO6): now also J5.4 (Pin_4)
- net at A1.13 (GPIO7): now also J5.5 (Pin_5)
- net at A1.14 (GPIO8): now also J5.6 (Pin_6)
- net at A1.15 (GPIO9): now also J5.7 (Pin_7)
- net at A1.16 (GPIO10): now also J5.8 (Pin_8)
- net at A1.6 (GPIO0): now also J3.1 (Pin_1)
- net at A1.7 (GPIO1): now also J3.2 (Pin_2)
- net at A1.8 (GPIO2): now also J3.3 (Pin_3)
- net at A1.9 (GPIO3): now also J5.1 (Pin_1)
- net +5V FILTERED renamed +5V
- net +5V: now also J6.2 (Pin_2)
- no-connect marks 32 -> 24
Other:
- moved on the sheet: C2, C5, J4, U1, U5
