File: hardware/neopico-hd/neopico-hd.kicad_pcb (KiCad board)
At the start: 2 copper layers, 24 parts, among them J1 HDMI_A, J2 Conn_02x05_Top_Bottom, J3 Conn_02x05_Top_Bottom, J4 Audio, U1 A_BUFF, U2 V_BUFF, U3 RG_LVS, U4 GB_LVS, U5 AV_LVS, U6 V_BUFF

Commit message: Update PCB
Parts:
- removed C8: 0.1u, Capacitor_SMD:C_0805_2012Metric_Pad1.18x1.45mm_HandSolder
- removed U6: V_BUFF, Package_TO_SOT_SMD:SOT-23-6
- added J5: AUX, Connector_JST:JST_XA_B08B-XASK-1_1x08_P2.50mm_Vertical, F.Cu at (139.4, 105.6)
- added J6: Conn_01x02_Pin, Connector_PinHeader_2.54mm:PinHeader_1x02_P2.54mm_Vertical, F.Cu at (181.9, 104.6)
- J2: footprint Connector_IDC:IDC-Header_2x05_P2.54mm_Vertical -> Connector_IDC:IDC-Header_2x10_P2.54mm_Vertical
- J3: value Conn_02x05_Top_Bottom -> Audio; footprint Connector_IDC:IDC-Header_2x05_P2.54mm_Vertical -> Connector_JST:JST_XA_B03B-XASK-1_1x03_P2.50mm_Vertical
- moved C7 67.4 mm to (173.0, 42.4), turned to 90 degrees
- moved C1 67.0 mm to (140.8, 95.8)
- moved REF** 66.8 mm to (150.4, 104.6)
- moved REF** 58.4 mm to (154.4, 104.6)
- moved U2 57.2 mm to (140.6, 92.4)
- moved C6 55.4 mm to (174.8, 104.6)
- moved D1 55.4 mm to (160.8, 104.6)
- moved F1 55.4 mm to (168.8, 106.1)
- moved FB1 55.4 mm to (168.8, 103.1)
- moved C2 55.1 mm to (148.0, 41.6), turned to 180 degrees
- moved C3 49.8 mm to (140.6, 55.2), turned to 180 degrees
- moved U3 48.5 mm to (140.7, 67.1)
- moved J2 48.5 mm to (123.5, 63.2)
- moved U1 47.3 mm to (140.6, 52.0)
- moved U5 47.1 mm to (140.8, 43.9)
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Connections:
- net +5V FILTERED renamed +5V
- A1 pad 10: unconnected-(A1-GPIO4-Pad10) -> Net-(A1-GPIO4)
- A1 pad 11: unconnected-(A1-GPIO5-Pad11) -> Net-(A1-GPIO5)
- A1 pad 12: unconnected-(A1-GPIO6-Pad12) -> Net-(A1-GPIO6)
- A1 pad 13: unconnected-(A1-GPIO7-Pad13) -> Net-(A1-GPIO7)
- A1 pad 14: unconnected-(A1-GPIO8-Pad14) -> Net-(A1-GPIO8)
- A1 pad 15: unconnected-(A1-GPIO9-Pad15) -> Net-(A1-GPIO9)
- A1 pad 16: unconnected-(A1-GPIO10-Pad16) -> Net-(A1-GPIO10)
- A1 pad 3: unconnected-(A1-AGND-Pad3) -> GND
- A1 pad 33: unconnected-(A1-GPIO27-Pad33) -> CSYNC
- A1 pad 34: unconnected-(A1-GPIO28-Pad34) -> PCKL
- A1 pad 35: PCKL -> B4
- A1 pad 36: CSYNC -> B3
- A1 pad 37: SHD -> B2
- A1 pad 38: DARK -> B1
- A1 pad 39: B4 -> B0
- A1 pad 4: unconnected-(A1-AGND-Pad4) -> GND
- A1 pad 40: B3 -> G4
- A1 pad 41: B2 -> G3
- A1 pad 42: B1 -> G2
- A1 pad 43: B0 -> G1
- A1 pad 44: G4 -> G0
- A1 pad 45: G3 -> R4
- A1 pad 47: G1 -> R2
- A1 pad 48: G0 -> R1
- A1 pad 49: (no net) -> R0
- A1 pad 50: R4 -> SHD
- A1 pad 51: R3 -> DARK
- A1 pad 52: R2 -> unconnected-(A1-GPIO46-Pad52)
- A1 pad 53: R1 -> unconnected-(A1-GPIO47-Pad53)
- A1 pad 54: R0 -> (no net)
- A1 pad 57: unconnected-(A1-AGND-Pad57) -> GND
- A1 pad 59: unconnected-(A1-AGND-Pad59) -> GND
- A1 pad 6: unconnected-(A1-GPIO0-Pad6) -> Net-(A1-GPIO0)
- A1 pad 60: unconnected-(A1-AGND-Pad60) -> GND
- A1 pad 7: unconnected-(A1-GPIO1-Pad7) -> Net-(A1-GPIO1)
- A1 pad 8: unconnected-(A1-GPIO2-Pad8) -> Net-(A1-GPIO2)
- A1 pad 9: unconnected-(A1-GPIO3-Pad9) -> Net-(A1-GPIO3)
- J3 pad 1: MVS_B0 -> Net-(A1-GPIO0)
- J3 pad 2: MVS_B1 -> Net-(A1-GPIO1)
- J3 pad 3: MVS_B2 -> Net-(A1-GPIO2)
- U2 pad 1: MVS_PCKL -> MVS_CSYNC
- U2 pad 3: MVS_CSYNC -> MVS_PCKL
- U2 pad 4: CSYNC -> PCKL
- U2 pad 6: PCKL -> CSYNC
- U5 pad 11: unconnected-(U5-B8-Pad11) -> DARK
- U5 pad 12: unconnected-(U5-B7-Pad12) -> SHD
- U5 pad 8: unconnected-(U5-A7-Pad8) -> MVS_SHD
- U5 pad 9: unconnected-(U5-A8-Pad9) -> MVS_DARK
Routing:
- net +5V: track 5.67 -> 66.1 mm
- net SHD: track 0.00 -> 60.1 mm, vias 0 -> 1
- net DARK: track 0.00 -> 59.4 mm, vias 0 -> 1
- net GND: track 16.9 -> 75.7 mm, vias 0 -> 2
- net MVS_DARK: track 0.00 -> 45.1 mm, vias 0 -> 1
- net R1: track 0.00 -> 42.1 mm
- net MVS_SHD: track 0.00 -> 41.7 mm, vias 0 -> 1
- net R0: track 0.00 -> 40.6 mm
- net R3: track 0.00 -> 39.5 mm
- net R2: track 0.00 -> 37.9 mm
- net G0: track 0.00 -> 36.8 mm
- net R4: track 0.00 -> 35.2 mm
- net G2: track 0.00 -> 34.2 mm
- net G1: track 0.00 -> 32.6 mm
- net G4: track 0.00 -> 27.6 mm
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Other:
- board outline added: 70.1 x 72.2 mm
