File: hardware/neopico-hd/neopico-hd.kicad_pcb (KiCad board)
At the start: 2 copper layers, 70 x 73.1 mm, 37 parts, among them J1 HDMI_A, J5 AUX, J6 Conn_01x02_Pin, T1 TestPoint_Pad_D1.0mm, U1 A_BUFF, U2 V_BUFF, U3 RG_LVS, U4 GB_LVS, U5 AV_LVS

Commit message: Minor hardware tweaks
Parts:
- C6: footprint Capacitor_THT:CP_Radial_D5.0mm_P2.00mm -> Capacitor_SMD:CP_Elec_6.3x5.4_Nichicon
- F1: value Polyfuse -> MF-PSMF020X-2
- J2: renamed from Video In
- J4: renamed from Audio In; footprint Connector_JST:JST_XA_B03B-XASK-1_1x03_P2.50mm_Vertical -> Connector_JST:JST_XA_B04B-XASK-1_1x04_P2.50mm_Vertical
- SW1: renamed from MENU; footprint Button_Switch_SMD:SW_SPST_B3U-1000P -> Button_Switch_SMD:SW_SPST_CK_KXT3
- SW2: renamed from BACK; footprint Button_Switch_SMD:SW_SPST_B3U-1000P -> Button_Switch_SMD:SW_SPST_CK_KXT3
- U1: value A_BUFF -> SN74LVC2G14DBV
- U2: value V_BUFF -> SN74LVC2G14DBV
- U3: value RG_LVS -> SN74LVC245APW
- U4: value GB_LVS -> SN74LVC245APW
- U5: value AV_LVS -> SN74LVC245APW
- moved J4 2.54 mm to (121.7, 48.7)
- moved J6 2.51 mm to (181.8, 102.5), turned to -90 degrees
- moved F1 1.22 mm to (165.0, 104.1)
- moved FB1 1.22 mm to (165.0, 101.1)
- moved Power In 1.22 mm to (150.0, 102.5)
- moved C6 0.28 mm to (172.5, 102.6)
- moved D1 0.13 mm to (158.1, 102.6)
- renumbered RP2350 to A1
Connections:
- A1 pad 51: unconnected-(A1-GPIO45-Pad51) -> MVS_DARK
- J2 pad 17: unconnected-(J2-Pin_17-Pad17) -> MVS_DARK
- J2 pad 20: unconnected-(J2-Pin_20-Pad20) -> GND
- J4 pad 1: MVS_BCK -> GND
- J4 pad 2: MVS_WS -> MVS_BCK
- J4 pad 3: MVS_DAT -> MVS_WS
Routing:
- net MVS_DARK: track 0.00 -> 62.0 mm
- net +5V MVS: track 9.53 -> 10.6 mm
- net Net-(D1-K): track 5.67 -> 4.59 mm
- net GND: track 25.3 -> 24.5 mm, vias 19 -> 20
Other:
- board text removed: "C6"
